Commit message: new changes added

File: p3at_description/urdf/pioneer3at.urdf.xacro (robot description, xacro)
@@ -8,10 +8,18 @@
   <xacro:include filename="$(find p3at_description)/urdf/pioneer3at_body.xacro"/>
   <xacro:include filename="$(find p3at_description)/urdf/hokuyo_utm30lx.urdf.xacro"/>
+  <xacro:include filename="$(find p3at_description)/urdf/normal_camera.urdf.xacro" />
+  <xacro:include filename="$(find p3at_description)/urdf/imu.urdf.xacro" />
+  <!--
   <xacro:include filename="$(find p3at_description)/urdf/asus_camera.urdf.xacro" />
-  <xacro:hokuyo_utm30lx name="hokuyo" parent="base_link" ros_topic="hokuyo" update_rate="30" ray_count="1040" min_angle="130" max_angle="-130" >
-    <origin xyz="0.13 0 0.32" rpy="0 0 0"/>
+  -->
+  <xacro:hokuyo_utm30lx name="hokuyo" parent="base_link" ros_topic="hokuyo" update_rate="30" ray_count="1080" min_angle="-135" max_angle="135" >
+    <origin xyz="0.13 0 0.42" rpy="0 0 0"/>
   </xacro:hokuyo_utm30lx>
   <xacro:asus_camera name="camera" parent="base_link">
-	                <origin xyz="0.065 0.0 0.43" rpy="0 0 0"/>
+	<!-- <origin xyz="0.065 0.0 0.53" rpy="0.52359877559 0 0"/> -->
+	<!-- camera 30 derece yamuk takilirsa FC-->
+	<origin xyz="0.065 0.0 0.53" rpy="0 0 0"/> <!-- 30 -> 0.52359877559 45-> 0.7854 -->
   </xacro:asus_camera>
+  <xacro:imu name="imu_link" parent="base_link" topic="imu_data">
+  </xacro:imu>
 </robot>

File: p3at_description/urdf/pioneer3at_body.xacro (robot description, xacro)
@@ -155,4 +155,8 @@
       <odometryFrame>odom</odometryFrame>
       <broadcastTF>true</broadcastTF>
+      <a1>0.1</a1>
+      <a2>0.1</a2>
+      <a3>0.1</a3>
+      <a4>0.1</a4>
     </plugin>
   </gazebo>

Commit message: added 30 degree bend over camera

File: p3at_description/urdf/pioneer3at.urdf.xacro (robot description, xacro)
@@ -19,5 +19,5 @@
 	<!-- <origin xyz="0.065 0.0 0.53" rpy="0.52359877559 0 0"/> -->
 	<!-- camera 30 derece yamuk takilirsa FC-->
-	<origin xyz="0.065 0.0 0.53" rpy="0 0 0"/> <!-- 30 -> 0.52359877559 45-> 0.7854 -->
+	<origin xyz="0.065 0.0 0.53" rpy="0 52359877559 0"/> <!-- 30 -> 0.52359877559 45-> 0.7854 -->
   </xacro:asus_camera>
   <xacro:imu name="imu_link" parent="base_link" topic="imu_data">

Commit message: added bended camera 30 degree

File: p3at_description/urdf/pioneer3at.urdf.xacro (robot description, xacro)
@@ -19,5 +19,5 @@
 	<!-- <origin xyz="0.065 0.0 0.53" rpy="0.52359877559 0 0"/> -->
 	<!-- camera 30 derece yamuk takilirsa FC-->
-	<origin xyz="0.065 0.0 0.53" rpy="0 52359877559 0"/> <!-- 30 -> 0.52359877559 45-> 0.7854 -->
+	<origin xyz="0.065 0.0 0.53" rpy="0 0.52359877559 0"/> <!-- 30 -> 0.52359877559 45-> 0.7854 -->
   </xacro:asus_camera>
   <xacro:imu name="imu_link" parent="base_link" topic="imu_data">

Commit message: default version set

File: p3at_description/urdf/pioneer3at.urdf.xacro (robot description, xacro)
@@ -19,5 +19,5 @@
 	<!-- <origin xyz="0.065 0.0 0.53" rpy="0.52359877559 0 0"/> -->
 	<!-- camera 30 derece yamuk takilirsa FC-->
-	<origin xyz="0.065 0.0 0.53" rpy="0 0.52359877559 0"/> <!-- 30 -> 0.52359877559 45-> 0.7854 -->
+	<origin xyz="0.065 0.0 0.53" rpy="0 0 0"/> <!-- 30 -> 0.52359877559 45-> 0.7854 -->
   </xacro:asus_camera>
   <xacro:imu name="imu_link" parent="base_link" topic="imu_data">

Commit message: changed position of hokuyo

File: p3at_description/urdf/pioneer3at.urdf.xacro (robot description, xacro)
@@ -8,18 +8,18 @@
   <xacro:include filename="$(find p3at_description)/urdf/pioneer3at_body.xacro"/>
   <xacro:include filename="$(find p3at_description)/urdf/hokuyo_utm30lx.urdf.xacro"/>
-  <xacro:include filename="$(find p3at_description)/urdf/normal_camera.urdf.xacro" />
-  <xacro:include filename="$(find p3at_description)/urdf/imu.urdf.xacro" />
+  <!-- <xacro:include filename="$(find p3at_description)/urdf/normal_camera.urdf.xacro" /> -->
+  <!-- <xacro:include filename="$(find p3at_description)/urdf/imu.urdf.xacro" /> -->
   <!--
   <xacro:include filename="$(find p3at_description)/urdf/asus_camera.urdf.xacro" />
   -->
   <xacro:hokuyo_utm30lx name="hokuyo" parent="base_link" ros_topic="hokuyo" update_rate="30" ray_count="1080" min_angle="-135" max_angle="135" >
-    <origin xyz="0.13 0 0.42" rpy="0 0 0"/>
+    <origin xyz="0 0 0.70" rpy="0 0 0"/>
   </xacro:hokuyo_utm30lx>
-  <xacro:asus_camera name="camera" parent="base_link">
+  <!-- <xacro:asus_camera name="camera" parent="base_link"> -->
 	<!-- <origin xyz="0.065 0.0 0.53" rpy="0.52359877559 0 0"/> -->
 	<!-- camera 30 derece yamuk takilirsa FC-->
-	<origin xyz="0.065 0.0 0.53" rpy="0 0 0"/> <!-- 30 -> 0.52359877559 45-> 0.7854 -->
-  </xacro:asus_camera>
-  <xacro:imu name="imu_link" parent="base_link" topic="imu_data">
-  </xacro:imu>
+	<!-- <origin xyz="0.065 0.0 0.53" rpy="0 0 0"/> 30 -> 0.52359877559 45-> 0.7854 -->
+  <!-- </xacro:asus_camera>   -->
+  <!-- <xacro:imu name="imu_link" parent="base_link" topic="imu_data"> -->
+  <!-- </xacro:imu>  -->
 </robot>

Commit message: lidar height is reduced

File: p3at_description/urdf/pioneer3at.urdf.xacro (robot description, xacro)
@@ -14,5 +14,5 @@
   -->
   <xacro:hokuyo_utm30lx name="hokuyo" parent="base_link" ros_topic="hokuyo" update_rate="30" ray_count="1080" min_angle="-135" max_angle="135" >
-    <origin xyz="0 0 0.70" rpy="0 0 0"/>
+    <origin xyz="0 0 0.40" rpy="0 0 0"/>
   </xacro:hokuyo_utm30lx>
   <!-- <xacro:asus_camera name="camera" parent="base_link"> -->

Commit message: p3at description added.

File: p3at_description/urdf/pioneer3at.urdf.xacro (robot description, xacro)
@@ -8,18 +8,18 @@
   <xacro:include filename="$(find p3at_description)/urdf/pioneer3at_body.xacro"/>
   <xacro:include filename="$(find p3at_description)/urdf/hokuyo_utm30lx.urdf.xacro"/>
-  <!-- <xacro:include filename="$(find p3at_description)/urdf/normal_camera.urdf.xacro" /> -->
-  <!-- <xacro:include filename="$(find p3at_description)/urdf/imu.urdf.xacro" /> -->
+  <xacro:include filename="$(find p3at_description)/urdf/normal_camera.urdf.xacro" />
+  <xacro:include filename="$(find p3at_description)/urdf/imu.urdf.xacro" />
   <!--
   <xacro:include filename="$(find p3at_description)/urdf/asus_camera.urdf.xacro" />
   -->
   <xacro:hokuyo_utm30lx name="hokuyo" parent="base_link" ros_topic="hokuyo" update_rate="30" ray_count="1080" min_angle="-135" max_angle="135" >
-    <origin xyz="0 0 0.40" rpy="0 0 0"/>
+    <origin xyz="0.13 0 0.42" rpy="0 0 0"/>
   </xacro:hokuyo_utm30lx>
-  <!-- <xacro:asus_camera name="camera" parent="base_link"> -->
+  <xacro:asus_camera name="camera" parent="base_link">
 	<!-- <origin xyz="0.065 0.0 0.53" rpy="0.52359877559 0 0"/> -->
 	<!-- camera 30 derece yamuk takilirsa FC-->
-	<!-- <origin xyz="0.065 0.0 0.53" rpy="0 0 0"/> 30 -> 0.52359877559 45-> 0.7854 -->
-  <!-- </xacro:asus_camera>   -->
-  <!-- <xacro:imu name="imu_link" parent="base_link" topic="imu_data"> -->
-  <!-- </xacro:imu>  -->
+	<origin xyz="0.065 0.0 0.53" rpy="0 0 0"/> <!-- 30 -> 0.52359877559 45-> 0.7854 -->
+  </xacro:asus_camera>
+  <xacro:imu name="imu_link" parent="base_link" topic="imu_data">
+  </xacro:imu>
 </robot>
